File: hardware/sensor-pcb/sensor-pcb.kicad_pcb (KiCad board)
At the start: 4 copper layers, 57 x 33 mm, 69 parts, among them J1 Conn_ARM_SWD_TagConnect_TC2030, J2 S5B-PH-SM4-TB, J4 S4B-PH-SM4-TB, Q1 BSS138BKSH, SW1 SKRKAHE020, SW2 SKRKAHE020, U1 STM32L476RCTx, U2 AP7354-33W5-7, U4 AP7354-33W5-7

Commit message: Changed trimmer back to JR200
Parts:
- C15: value JR030 -> JR200
Changed lines of the file:
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@@
 			)
 		)
-		(property "Value" "JR030"
+		(property "Value" "JR200"
 			(at 0 3 270)
 			(unlocked yes)
@@
 			)
 		)
-		(property "MFPN" "JR030"
+		(property "MFPN" "JR200"
 			(at 0 0 270)
 			(unlocked yes)
